Commit message: Added writing support. Axis are fines except for Y which is inverted. I don't understand how to put that correctly, i tried everything. World frame should be fixed on arm_base, and table placed depending on world/frame / arm_base.

File: kuka_lwr_description/robots/kuka_lwr_laas.urdf.xacro (robot description, xacro)
@@ -4,6 +4,6 @@
 	<xacro:include filename="$(find kuka_lwr_description)/defs/materials.xml"/>
 	<xacro:include filename="$(find kuka_lwr_description)/urdf/kuka_lwr_arm_laas.urdf.xacro"/> <!-- POSITIONNEMENT BRAS -->
-	<kuka_lwr_arm_laas parent="table_top_link" name="right">
-          <origin xyz="0.8 0.0 1.2" rpy="0 1.5708 3.14159"/>
+	<kuka_lwr_arm_laas parent="table_top_link" name="right"> <!-- On définit la position du bras par rapport a table_top_link sur lequel j'ai rattaché la world frame -->
+          <origin xyz="0.8 0.0 1.2" rpy="0 ${M_PI / 2} ${M_PI}"/>
         </kuka_lwr_arm_laas>
 </robot>

File: kuka_lwr_description/urdf/kuka_lwr_arm_laas.urdf.xacro (robot description, xacro)
@@ -146,4 +146,18 @@
    <link name="${name}_arm_flange_link">
    </link>
+    <link name="${name}_writting_support_link">
+      <visual>
+        <origin xyz="0.0 0 0.01" rpy="${M_PI} 0 0"/>
+        <geometry>
+          <mesh filename="package://kuka_lwr_description/meshes/writing_support.dae" scale="0.001 0.001 0.001"/>
+        </geometry>
+        <material name="Black"/>
+      </visual>
+    </link>
+   <joint name="${name}_writting_support_joint" type="fixed">
+      <origin xyz="0 0 0" rpy="0 0 0"/>
+      <parent link="${name}_arm_flange_link"/>
+      <child link="${name}_writting_support_link"/>
+   </joint>
   </macro>
 </robot>
